File: Sending end.sch (EAGLE design)
At the start: 17 parts, among them IC1 MEGA8-P, Q1 16 MHz

Commit message: polished schematic
Parts:
- removed C1, C2: 22pF, rcl:C-EUC1210
- removed D1: HSMXC670, opto-transmittter-hp:HSMXC670
- removed Q1: 16 MHz, crystal:CRYSTALHC49S
- removed S1: SWS001, smd-special:SWS001
- added R10, R6, R7, R8, R9: tbd, resistor:R-EU_M0805
Connections:
- removed net BRAKE: R5.1
- removed net LEFT_TURN: R4.1
- removed net N$4: IC1.PD5(T1), R2.2
- removed net N$9: D4.C, IC1.PC1(ADC1), R4.2
- removed net RIGHT_TURN: R3.1
- new net N$26: D3.C, IC1.PC0(ADC0), R1.2, R3.2, R6.2
- net GND: now also IC1.PB6(XTAL1/TOSC1); no longer C1.2, D1.C, Q1.1
- net N$1: now also IC1.PD3(INT1); no longer C1.1, C2.1
- net N$10: now also R5.1, R8.1, R9.1; no longer D5.C, IC1.PC2(ADC2), R5.2
- net N$2: now also D4.C, IC1.PC1(ADC1), R10.2, R4.2, R7.2; no longer C2.2, IC1.PB6(XTAL1/TOSC1), Q1.2
- net N$20: now also R2.2
- net N$3: now also D5.C, IC1.PC2(ADC2), R5.2, R8.2, R9.2; no longer IC1.PD3(INT1), R1.2
- net N$5: now also R3.1, R6.1; no longer D1.A
- net N$7: no longer S1.1
- net N$8: now also R10.1, R4.1, R7.1; no longer D3.C, IC1.PC0(ADC0), R3.2
- net VCC: no longer S1.2
Other:
- note removed: "_(+)12VDC Batt"
- note removed: "_(-)12VDC Batt"
- moved on the sheet: 12V-5VDCDCCONVERTER, D2, D3, D4, D5, R1, R2, R3, R4, R5
